File: BoardRover2/BoardRover2.kicad_pcb (KiCad board)
At the start: 2 copper layers, 82.1 x 88.9 mm, 37 parts, among them J1 Conn_01x06_Socket, J2 Conn_01x06_Socket, J3 Motor2, J4 Motor1, J5 10V, J6 Encoder1, J7 Encoder2, J8 Servo1, J9 Servo2, U1 PC817, U10 LM350_TO220, U11 YAAJ_BluePill_Part_Like, U2 PC817, U3 PC817, U5 AMS1117-5.0, U6 PC817, U7 PC817, U8 PC817, U9 YAAJ_BluePill_Part_Like

Commit message: LED Y FUSIL
Parts:
- added D1: LED, LED_THT:LED_D3.0mm_Clear, F.Cu at (212.5, 106.7)
- added D2: LED, LED_THT:LED_D3.0mm_Clear, F.Cu at (195.6, 61.0)
- added F1: Fuse, Fuse:Fuse_1812_4532Metric, B.Cu at (182.5, 121.5)
- added R11: 1KR, Resistor_SMD:R_1206_3216Metric, B.Cu at (213.2, 93.7)
- added R12: 1KR, Resistor_SMD:R_1206_3216Metric, B.Cu at (189.0, 61.0)
- moved R13 1.08 mm to (208.3, 78.3)
- moved R14 1.08 mm to (208.3, 88.5)
- moved R15 1.08 mm to (208.3, 99.1)
Connections:
- J1 pad 4: 10V -> Net-(J1-MotorVCC)
- U11 pad 39: unconnected-(U11-GND-Pad39) -> Net-(R12-Pad1)
Routing:
- net Net-(D1-A): track 0.00 -> 9.23 mm
- net 10V: track 40.0 -> 31.3 mm
- net Net-(R12-Pad1): track 0.00 -> 5.75 mm
- net 5V: track 217.9 -> 223.5 mm
- net Net-(J1-MotorVCC): track 0.00 -> 5.26 mm
- net Net-(D2-A): track 0.00 -> 2.54 mm
- net In3: track 49.5 -> 48.4 mm
- net In4: track 38.0 -> 36.9 mm

Commit message: doble board y correxion
Parts:
- moved F1 17.7 mm to (165.1, 124.9), turned to -90 degrees
- moved C1 5.81 mm to (171.4, 126.0)
- moved J5 5.72 mm to (166.6, 131.0)
Connections:
- F1 pad 1: Net-(J1-MotorVCC) -> 10V
- F1 pad 2: 10V -> Net-(J5-Pin_1)
- J1 pad 1: In4 -> In1
- J1 pad 2: In3 -> In2
- J1 pad 3: PowerGND -> 10V
- J1 pad 4: Net-(J1-MotorVCC) -> PowerGND
- J1 pad 5: In2 -> In3
- J1 pad 6: In1 -> In4
- J5 pad 1: 10V -> Net-(J5-Pin_1)
- R13 pad 1: In3 -> In2
- R14 pad 1: In4 -> In1
- R17 pad 1: In1 -> In4
- R18 pad 1: In2 -> In3
- U1 pad 4: In3 -> In2
- U2 pad 4: In4 -> In1
- U6 pad 4: In1 -> In4
- U7 pad 4: In2 -> In3
Routing:
- net In3: track 48.4 -> 73.6 mm
- net In2: track 73.6 -> 48.4 mm
- net In1: track 59.1 -> 36.9 mm
- net In4: track 36.9 -> 58.4 mm
- net 10V: track 31.3 -> 37.7 mm
- net 7V: track 102.7 -> 109.1 mm
- net Net-(J1-MotorVCC): track 5.26 -> 0.00 mm
- net Net-(J5-Pin_1): track 0.00 -> 4.66 mm
- net Out1: track 41.5 -> 43.6 mm
- net Out2: track 47.0 -> 49.1 mm
Other:
- board size 82.1 x 88.9 mm -> 82.1 x 91.4 mm
