File: BoardRover2/BoardRover2.kicad_sch (KiCad schematic)
At the start: 37 parts, among them J1 Conn_01x06_Socket, J2 Conn_01x06_Socket, J3 Motor2, J4 Motor1, J5 10V, J6 Encoder1, J7 Encoder2, J8 Servo1, J9 Servo2, U1 PC817, U10 LM350_TO220, U11 YAAJ_BluePill_Part_Like, U2 PC817, U3 PC817, U5 AMS1117-5.0, U6 PC817, U7 PC817, U8 PC817, U9 YAAJ_BluePill_Part_Like

Commit message: LED Y FUSIL
Parts:
- added D1, D2: LED, LED_THT:LED_D3.0mm_Clear, symbol Device:LED
- added F1: Fuse, Fuse:Fuse_1812_4532Metric, symbol Device:Fuse
- added R11, R12: 1KR, Resistor_SMD:R_1206_3216Metric, symbol Device:R
Connections:
- net 10V: now also F1.2; no longer J1.4 (MotorVCC)
- net 5V: now also R11.1
- net DGnd: now also D2.1 (K)
- net PowerGND: now also D1.1 (K)
- net at U11.39 (GND): now also R12.1
- new net: F1.1, J1.4 (MotorVCC)
- new net: D1.2 (A), R11.2
- new net: D2.2 (A), R12.2

Commit message: doble board y correxion
Connections:
- net 10V: now also F1.1, J1.3 (MotorGND); no longer F1.2, J5.1 (Pin_1)
- net In1: now also J1.1 (In4), R14.1, U2.4; no longer J1.6 (In1), R17.1, U6.4
- net In2: now also J1.2 (In3), R13.1, U1.4; no longer J1.5 (In2), R18.1, U7.4
- net In3: now also J1.5 (In2), R18.1, U7.4; no longer J1.2 (In3), R13.1, U1.4
- net In4: now also J1.6 (In1), R17.1, U6.4; no longer J1.1 (In4), R14.1, U2.4
- net PowerGND: now also J1.4 (MotorVCC); no longer J1.3 (MotorGND)
- new net: F1.2, J5.1 (Pin_1)
Other:
- moved on the sheet: C1, F1
Changed lines of the file:
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@@
 	)
 	(junction
-		(at 107.95 144.78)
+		(at 105.41 144.78)
 		(diameter 0)
 		(color 0 0 0 0)
@@
 	(wire
 		(pts
-			(xy 154.94 50.8) (xy 156.21 50.8)
+			(xy 101.6 144.78) (xy 105.41 144.78)
 		)
 		(stroke
@@
 	(wire
 		(pts
-			(xy 161.29 68.58) (xy 166.37 68.58)
+			(xy 154.94 50.8) (xy 156.21 50.8)
 		)
 		(stroke
@@
 	(wire
 		(pts
-			(xy 167.64 163.83) (xy 167.64 166.37)
+			(xy 161.29 68.58) (xy 166.37 68.58)
 		)
 		(stroke
@@
 	(wire
 		(pts
-			(xy 128.27 144.78) (xy 130.81 144.78)
+			(xy 167.64 163.83) (xy 167.64 166.37)
 		)
 		(stroke
@@
 	(wire
 		(pts
-			(xy 143.51 144.78) (xy 151.13 144.78)
+			(xy 128.27 144.78) (xy 130.81 144.78)
 		)
 		(stroke
@@
 	(wire
 		(pts
-			(xy 137.16 121.92) (xy 146.05 121.92)
+			(xy 143.51 144.78) (xy 151.13 144.78)
 		)
 		(stroke
@@
 	(wire
 		(pts
-			(xy 104.14 144.78) (xy 107.95 144.78)
-		)
-		(stroke
-			(width 0)
-			(type default)
-		)
-	)
-	(wire
-		(pts
 			(xy 205.74 68.58) (xy 208.28 68.58)
 		)
@@
 	(wire
 		(pts
-			(xy 107.95 144.78) (xy 113.03 144.78)
-		)
-		(stroke
-			(width 0)
-			(type default)
-		)
-	)
-	(wire
-		(pts
 			(xy 86.36 115.57) (xy 97.79 115.57)
 		)
@@
 	(wire
 		(pts
-			(xy 107.95 144.78) (xy 107.95 147.32)
+			(xy 105.41 144.78) (xy 105.41 147.32)
 		)
 		(stroke
@@
 	(wire
 		(pts
+			(xy 105.41 144.78) (xy 113.03 144.78)
+		)
+		(stroke
+			(width 0)
+			(type default)
+		)
+	)
+	(wire
+		(pts
 			(xy 114.3 73.66) (xy 102.87 73.66)
 		)
@@
 	(wire
 		(pts
-			(xy 160.02 38.1) (xy 160.02 35.56)
+			(xy 137.16 124.46) (xy 140.97 124.46)
 		)
 		(stroke
@@
 	(wire
 		(pts
-			(xy 166.37 144.78) (xy 167.64 144.78)
+			(xy 160.02 38.1) (xy 160.02 35.56)
 		)
 		(stroke
@@
 	(wire
 		(pts
-			(xy 102.87 73.66) (xy 102.87 63.5)
+			(xy 166.37 144.78) (xy 167.64 144.78)
 		)
 		(stroke
@@
 	(wire
 		(pts
-			(xy 167.64 144.78) (xy 167.64 146.05)
+			(xy 102.87 73.66) (xy 102.87 63.5)
 		)
 		(stroke
@@
 	(wire
 		(pts
-			(xy 83.82 68.58) (xy 88.9 68.58)
+			(xy 167.64 144.78) (xy 167.64 146.05)
 		)
 		(stroke
@@
 	(wire
 		(pts
-			(xy 153.67 121.92) (xy 160.02 121.92)
+			(xy 83.82 68.58) (xy 88.9 68.58)
 		)
 		(stroke
@@
 	(global_label "10V"
 		(shape input)
-		(at 160.02 121.92 0)
+		(at 140.97 124.46 0)
 		(effects
 			(font
@@
 		)
 		(property "Intersheetrefs" "${INTERSHEET_REFS}"
-			(at 160.02 121.92 0)
+			(at 140.97 124.46 0)
 			(effects
 				(font
@@
 		)
 	)
-	(global_label "In1"
-		(shape input)
-		(at 137.16 116.84 0)
-		(effects
-			(font
-				(size 1.27 1.27)
-			)
-			(justify left)
-		)
-		(property "Intersheetrefs" "${INTERSHEET_REFS}"
-			(at 137.16 116.84 0)
-			(effects
-				(font
-					(size 1.27 1.27)
-				)
-				(hide yes)
-			)
-		)
-	)
 	(global_label "PB9"
 		(shape input)
@@
 		)
 	)
-	(global_label "In1"
+	(global_label "In4"
 		(shape input)
 		(at 63.5 44.45 90)
@@
 		)
 	)
-	(global_label "In2"
+	(global_label "In3"
 		(shape input)
 		(at 137.16 119.38 0)
@@
 	(global_label "PowerGND"
 		(shape input)
-		(at 137.16 124.46 0)
+		(at 137.16 121.92 0)
 		(effects
 			(font
@@
 		)
 		(property "Intersheetrefs" "${INTERSHEET_REFS}"
-			(at 137.16 124.46 0)
+			(at 137.16 121.92 0)
 			(effects
 				(font
@@
 		)
 	)
-	(global_label "In3"
+	(global_label "In2"
 		(shape input)
 		(at 195.58 49.53 90)
@@
 		)
 	)
-	(global_label "In4"
+	(global_label "In1"
 		(shape input)
 		(at 195.58 66.04 90)
@@
 		)
 	)
-	(global_label "In2"
+	(global_label "In3"
 		(shape input)
 		(at 63.5 59.69 90)
@@
 	(global_label "PowerGND"
 		(shape input)
-		(at 107.95 154.94 270)
+		(at 105.41 154.94 270)
 		(fields_autoplaced yes)
 		(effects
@@
 		)
 		(property "Intersheetrefs" "${INTERSHEET_REFS}"
-			(at 107.95 167.42 90)
+			(at 105.41 167.42 90)
 			(effects
 				(font
@@
 	(global_label "10V"
 		(shape input)
-		(at 82.55 147.32 180)
+		(at 74.93 147.32 180)
 		(fields_autoplaced yes)
 		(effects
@@
 		)
 		(property "Intersheetrefs" "${INTERSHEET_REFS}"
-			(at 76.0572 147.32 0)
+			(at 68.4372 147.32 0)
 			(effects
 				(font
@@
 		)
 	)
-	(global_label "In3"
+	(global_label "In2"
 		(shape input)
 		(at 137.16 127 0)
@@
 		)
 	)
-	(global_label "In1"
+	(global_label "In4"
 		(shape input)
 		(at 137.16 116.84 0)
@@
 		)
 	)
-	(global_label "In4"
+	(global_label "In1"
 		(shape input)
 		(at 137.16 129.54 0)
@@
 	(global_label "10V"
 		(shape input)
-		(at 104.14 144.78 180)
+		(at 101.6 144.78 180)
 		(fields_autoplaced yes)
 		(effects
@@
 		)
 		(property "Intersheetrefs" "${INTERSHEET_REFS}"
-			(at 97.6472 144.78 0)
+			(at 95.1072 144.78 0)
 			(effects
 				(font
@@
 	(symbol
 		(lib_id "Device:Fuse")
-		(at 149.86 121.92 90)
+		(at 78.74 147.32 90)
 		(unit 1)
 		(exclude_from_sim no)
@@
 		(on_board yes)
 		(dnp no)
-		(fields_autoplaced yes)
 		(property "Reference" "F1"
-			(at 149.86 115.57 90)
+			(at 77.724 144.78 90)
 			(effects
 				(font
@@
 		)
 		(property "Value" "Fuse"
-			(at 149.86 118.11 90)
+			(at 82.296 144.018 90)
 			(effects
 				(font
@@
 		)
 		(property "Footprint" "Fuse:Fuse_1812_4532Metric"
-			(at 149.86 123.698 90)
+			(at 78.74 149.098 90)
 			(effects
 				(font
@@
 		)
 		(property "Datasheet" "~"
-			(at 149.86 121.92 0)
+			(at 78.74 147.32 0)
 			(effects
 				(font
@@
 		)
 		(property "Description" "Fuse"
-			(at 149.86 121.92 0)
+			(at 78.74 147.32 0)
 			(effects
 				(font
@@
 		)
 		(instances
-			(project ""
+			(project "BoardRover2"
 				(path "/d68abd69-b3fe-45ee-a6d1-5f3c4ed0dd64"
 					(reference "F1")
@@
 	(symbol
 		(lib_id "Device:C_Polarized")
-		(at 107.95 151.13 0)
+		(at 105.41 151.13 0)
 		(unit 1)
 		(exclude_from_sim no)
@@
 		(dnp no)
 		(property "Reference" "C1"
-			(at 110.998 150.876 0)
+			(at 108.458 150.876 0)
 			(effects
 				(font
@@
 		)
 		(property "Value" "10uF"
-			(at 100.584 151.13 0)
+			(at 98.044 151.13 0)
 			(effects
 				(font
@@
 		)
 		(property "Footprint" "Capacitor_SMD:C_1206_3216Metric"
-			(at 108.9152 154.94 0)
+			(at 106.3752 154.94 0)
 			(effects
 				(font
@@
 		)
 		(property "Datasheet" "~"
-			(at 107.95 151.13 0)
+			(at 105.41 151.13 0)
 			(effects
 				(font
@@
 		)
 		(property "Description" "Polarized capacitor"
-			(at 107.95 151.13 0)
+			(at 105.41 151.13 0)
 			(effects
 				(font
